Commit message: PR06 defect: attach lidar to camera instead of base (do not merge)
Co-Authored-By: Claude Code <noreply@anthropic.com>

File: src/course_description/urdf/vehicle.urdf.xacro (robot description, xacro)
@@ -85,5 +85,5 @@
   </link>
   <joint name="lidar_joint" type="fixed">
-    <parent link="base_link"/><child link="lidar_link"/>
+    <parent link="camera_link"/><child link="lidar_link"/>
     <origin xyz="0.28 0 0.38"/>
   </joint>
